Commit message: Every link has a small sphere as a visual object at its center

File: horse_based_robot.urdf (robot description, URDF)
Before this commit: robot a1, 28 links, 27 joints
Links:
- link Ears: geometry visual sphere radius=0.01
- link FL_calf: geometry collision box size=0.2 0.016 0.016; visual sphere radius=0.01
- link FL_hip: geometry collision cylinder length=0.04 radius=0.046; visual sphere radius=0.01
- link FL_pre_hip: geometry visual sphere radius=0.01
- link FL_thigh: geometry collision box size=0.2 0.0245 0.034; visual sphere radius=0.01
- link FR_calf: geometry collision box size=0.2 0.016 0.016; visual sphere radius=0.01
- link FR_hip: geometry collision cylinder length=0.04 radius=0.046; visual sphere radius=0.01
- link FR_pre_hip: geometry visual sphere radius=0.01
- link FR_thigh: geometry collision box size=0.2 0.0245 0.034; visual sphere radius=0.01
- link Jawline: geometry visual sphere radius=0.01
- link Lower Spine: geometry visual sphere radius=0.01
- link Nose: geometry visual sphere radius=0.01
- link RL_calf: geometry collision box size=0.2 0.016 0.016; visual sphere radius=0.01
- link RL_hip: geometry collision cylinder length=0.04 radius=0.046; visual sphere radius=0.01
- link RL_pre_hip: geometry visual sphere radius=0.01
- link RL_thigh: geometry collision box size=0.2 0.0245 0.034; visual sphere radius=0.01
- link RR_calf: geometry collision box size=0.2 0.016 0.016; visual sphere radius=0.01
- link RR_hip: geometry collision cylinder length=0.04 radius=0.046; visual sphere radius=0.01
- link RR_pre_hip: geometry visual sphere radius=0.01
- link RR_thigh: geometry collision box size=0.2 0.0245 0.034; visual sphere radius=0.01
- link Tail: geometry visual sphere radius=0.01
- link Upper Spine: geometry visual sphere radius=0.01
- link base: geometry visual sphere radius=0.01
- link trunk: geometry collision box size=0.267 0.194 0.114; visual sphere radius=0.01

Commit message: Checkpoint

File: horse_based_robot.urdf (robot description, URDF)
Before this commit: robot a1, 28 links, 27 joints
Links:
- link Ears: geometry visual sphere radius=0.1
- link FL_calf: geometry collision box size=0.2 0.016 0.016; visual sphere radius=0.1
- link FL_foot: geometry collision sphere radius=0.02; visual sphere radius=0.1
- link FL_hip: geometry collision cylinder length=0.04 radius=0.046; visual sphere radius=0.1
- link FL_pre_hip: geometry visual sphere radius=0.1
- link FL_thigh: geometry collision box size=0.2 0.0245 0.034; visual sphere radius=0.1
- link FR_calf: geometry collision box size=0.2 0.016 0.016; visual sphere radius=0.1
- link FR_foot: geometry collision sphere radius=0.02; visual sphere radius=0.1
- link FR_hip: geometry collision cylinder length=0.04 radius=0.046; visual sphere radius=0.1
- link FR_pre_hip: geometry visual sphere radius=0.1
- link FR_thigh: geometry collision box size=0.2 0.0245 0.034; visual sphere radius=0.1
- link Jawline: geometry visual sphere radius=0.1
- link Lower Spine: geometry visual sphere radius=0.1
- link Nose: geometry visual sphere radius=0.1
- link RL_calf: geometry collision box size=0.2 0.016 0.016; visual sphere radius=0.1
- link RL_foot: geometry collision sphere radius=0.02; visual sphere radius=0.1
- link RL_hip: geometry collision cylinder length=0.04 radius=0.046; visual sphere radius=0.1
- link RL_pre_hip: geometry visual sphere radius=0.1
- link RL_thigh: geometry collision box size=0.2 0.0245 0.034; visual sphere radius=0.1
- link RR_calf: geometry collision box size=0.2 0.016 0.016; visual sphere radius=0.1
- link RR_foot: geometry collision sphere radius=0.02; visual sphere radius=0.1
- link RR_hip: geometry collision cylinder length=0.04 radius=0.046; visual sphere radius=0.1
- link RR_pre_hip: geometry visual sphere radius=0.1
- link RR_thigh: geometry collision box size=0.2 0.0245 0.034; visual sphere radius=0.1
- link Tail: geometry visual sphere radius=0.1
- link Upper Spine: geometry visual sphere radius=0.1
- link base: geometry visual sphere radius=0.1
- link trunk: geometry collision box size=0.267 0.194 0.114; visual sphere radius=0.1
Joints:
- joint Craniovertebral Junction: origin xyz=113.6170 -2.5109 75.6393 rpy=0 0 0 -> xyz=1.1361700000000001 -0.025109 0.7563930000000001 rpy=0 0 0
- joint FL_calf_joint: origin xyz=-5.4575 0.6502 -53.3053 rpy=0 0 0 -> xyz=-0.054575 0.006502 -0.533053 rpy=0 0 0
- joint FL_foot_fixed: origin xyz=-8.8321 -1.0051 -45.4922 rpy=0 0 0 -> xyz=-0.08832100000000001 -0.010051000000000001 -0.454922 rpy=0 0 0
- joint FL_hip_joint: origin xyz=0.0000 0.0000 0.0000 rpy=0 0 0 -> xyz=0.0 0.0 0.0 rpy=0 0 0
- joint FL_pre_hip_joint: origin xyz=72.8557 19.1179 -96.7309 rpy=0 0 0 -> xyz=0.728557 0.191179 -0.9673090000000001 rpy=0 0 0
- joint FL_thigh_joint: origin xyz=0.0000 0.0000 0.0000 rpy=0 0 0 -> xyz=0.0 0.0 0.0 rpy=0 0 0
- joint FR_calf_joint: origin xyz=-5.4576 0.6502 -53.3053 rpy=0 0 0 -> xyz=-0.054576 0.006502 -0.533053 rpy=0 0 0
- joint FR_foot_fixed: origin xyz=-8.8321 -1.0051 -45.4922 rpy=0 0 0 -> xyz=-0.08832100000000001 -0.010051000000000001 -0.454922 rpy=0 0 0
- joint FR_hip_joint: origin xyz=0.0000 0.0000 0.0000 rpy=0 0 0 -> xyz=0.0 0.0 0.0 rpy=0 0 0
- joint FR_pre_hip_joint: origin xyz=90.2915 -24.6175 -95.3342 rpy=0 0 0 -> xyz=0.902915 -0.246175 -0.9533419999999999 rpy=0 0 0
- joint FR_thigh_joint: origin xyz=0.0000 0.0000 0.0000 rpy=0 0 0 -> xyz=0.0 0.0 0.0 rpy=0 0 0
- joint Jaw: origin xyz=-57.9458 1.2806 1.1844 rpy=0 0 0 -> xyz=-0.579458 0.012806 0.011843999999999999 rpy=0 0 0
- joint RL_calf_joint: origin xyz=-34.6984 1.2964 -70.9206 rpy=0 0 0 -> xyz=-0.346984 0.012964 -0.7092059999999999 rpy=0 0 0
- joint RL_foot_fixed: origin xyz=3.0974 -1.2687 -45.4922 rpy=0 0 0 -> xyz=0.030973999999999998 -0.012686999999999999 -0.454922 rpy=0 0 0
- joint RL_hip_joint: origin xyz=0.0000 0.0000 0.0000 rpy=0 0 0 -> xyz=0.0 0.0 0.0 rpy=0 0 0
- joint RL_pre_hip_joint: origin xyz=-56.4942 21.9765 -79.1156 rpy=0 0 0 -> xyz=-0.5649419999999999 0.21976500000000002 -0.791156 rpy=0 0 0
- joint RL_thigh_joint: origin xyz=0.0000 0.0000 0.0000 rpy=0 0 0 -> xyz=0.0 0.0 0.0 rpy=0 0 0
- joint RR_calf_joint: origin xyz=-44.8519 0.6079 -72.6681 rpy=0 0 0 -> xyz=-0.448519 0.006079 -0.7266809999999999 rpy=0 0 0
- joint RR_foot_fixed: origin xyz=-7.5565 3.3491 -44.6550 rpy=0 0 0 -> xyz=-0.075565 0.033491 -0.44655 rpy=0 0 0
- joint RR_hip_joint: origin xyz=0.0000 0.0000 0.0000 rpy=0 0 0 -> xyz=0.0 0.0 0.0 rpy=0 0 0
- joint RR_pre_hip_joint: origin xyz=-82.6344 -18.0470 -81.8491 rpy=0 0 0 -> xyz=-0.826344 -0.18047000000000002 -0.8184910000000001 rpy=0 0 0
- joint RR_thigh_joint: origin xyz=0.0000 0.0000 0.0000 rpy=0 0 0 -> xyz=0.0 0.0 0.0 rpy=0 0 0
- joint Spinal Midpoint Lower: origin xyz=-56.2901 1.2440 0.0000 rpy=0 0 0 -> xyz=-0.562901 0.01244 0.0 rpy=0 0 0
- joint Spinal Midpoint Upper: origin xyz=49.4218 -1.0922 0.0000 rpy=0 0 0 -> xyz=0.494218 -0.010922000000000001 0.0 rpy=0 0 0
- joint Start of Tail: origin xyz=-90.6485 2.0033 -73.2124 rpy=0 0 0 -> xyz=-0.906485 0.020033 -0.732124 rpy=0 0 0
- joint Top of Nose: origin xyz=57.0513 -1.2608 -52.1657 rpy=0 0 0 -> xyz=0.5705129999999999 -0.012608 -0.521657 rpy=0 0 0
- joint floating_base: origin xyz=0.0000 0.0000 0.0000 rpy=0 0 0 -> xyz=0.0 0.0 0.0 rpy=0 0 0

Commit message: Checkpoint

File: horse_based_robot.urdf (robot description, URDF)
Before this commit: robot a1, 28 links, 27 joints
Links:
- removed link FL_pre_hip
- removed link FR_pre_hip
- removed link RL_pre_hip
- removed link RR_pre_hip
- link Ears: geometry 
- link FL_calf: geometry collision box size=0.2 0.016 0.016; visual mesh filename=package://a1_description/meshes/calf.dae scale=1 1 1
- link FL_foot: geometry collision sphere radius=0.02; visual sphere radius=0.01
- link FL_hip: geometry collision cylinder length=0.04 radius=0.046; visual mesh filename=package://a1_description/meshes/hip.dae scale=1 1 1
- link FL_thigh: geometry collision box size=0.2 0.0245 0.034; visual mesh filename=package://a1_description/meshes/thigh.dae scale=1 1 1
- link FR_calf: geometry collision box size=0.2 0.016 0.016; visual mesh filename=package://a1_description/meshes/calf.dae scale=1 1 1
- link FR_foot: geometry collision sphere radius=0.02; visual sphere radius=0.01
- link FR_hip: geometry collision cylinder length=0.04 radius=0.046; visual mesh filename=package://a1_description/meshes/hip.dae scale=1 1 1
- link FR_thigh: geometry collision box size=0.2 0.0245 0.034; visual mesh filename=package://a1_description/meshes/thigh_mirror.dae scale=1 1 1
- link Jawline: geometry 
- link Lower Spine: geometry 
- link Nose: geometry 
- link RL_calf: geometry collision box size=0.2 0.016 0.016; visual mesh filename=package://a1_description/meshes/calf.dae scale=1 1 1
- link RL_foot: geometry collision sphere radius=0.02; visual sphere radius=0.01
- link RL_hip: geometry collision cylinder length=0.04 radius=0.046; visual mesh filename=package://a1_description/meshes/hip.dae scale=1 1 1
- link RL_thigh: geometry collision box size=0.2 0.0245 0.034; visual mesh filename=package://a1_description/meshes/thigh.dae scale=1 1 1
- link RR_calf: geometry collision box size=0.2 0.016 0.016; visual mesh filename=package://a1_description/meshes/calf.dae scale=1 1 1
- link RR_foot: geometry collision sphere radius=0.02; visual sphere radius=0.01
- link RR_hip: geometry collision cylinder length=0.04 radius=0.046; visual mesh filename=package://a1_description/meshes/hip.dae scale=1 1 1
- link RR_thigh: geometry collision box size=0.2 0.0245 0.034; visual mesh filename=package://a1_description/meshes/thigh_mirror.dae scale=1 1 1
- link Tail: geometry 
- link Upper Spine: geometry 
- link base: geometry visual box size=0.001 0.001 0.001
- link trunk: geometry collision box size=0.267 0.194 0.114; visual mesh filename=package://a1_description/meshes/trunk.dae scale=1 1 1
Joints:
- removed joint FL_pre_hip_joint
- removed joint FR_pre_hip_joint
- removed joint RL_pre_hip_joint
- removed joint RR_pre_hip_joint
- joint Craniovertebral Junction: origin xyz=1.1361700000000001 -0.025109 0.7563930000000001 rpy=0 0 0 -> xyz=113.6170 -2.5109 75.6393 rpy=0 0 0
- joint FL_calf_joint: origin xyz=-0.054575 0.006502 -0.533053 rpy=0 0 0 -> xyz=-5.4575 0.6502 -53.3053 rpy=0 0 0
- joint FL_foot_fixed: origin xyz=-0.08832100000000001 -0.010051000000000001 -0.454922 rpy=0 0 0 -> xyz=-8.8321 -1.0051 -45.4922 rpy=0 0 0
- joint FL_hip_joint: origin xyz=0.0 0.0 0.0 rpy=0 0 0 -> xyz=72.8557 19.1179 -96.7309 rpy=0 0 0; parent FL_pre_hip -> trunk
- joint FL_thigh_joint: origin xyz=0.0 0.0 0.0 rpy=0 0 0 -> xyz=0.0000 0.0000 0.0000 rpy=0 0 0
- joint FR_calf_joint: origin xyz=-0.054576 0.006502 -0.533053 rpy=0 0 0 -> xyz=-5.4576 0.6502 -53.3053 rpy=0 0 0
- joint FR_foot_fixed: origin xyz=-0.08832100000000001 -0.010051000000000001 -0.454922 rpy=0 0 0 -> xyz=-8.8321 -1.0051 -45.4922 rpy=0 0 0
- joint FR_hip_joint: origin xyz=0.0 0.0 0.0 rpy=0 0 0 -> xyz=90.2915 -24.6175 -95.3342 rpy=0 0 0; parent FR_pre_hip -> trunk
- joint FR_thigh_joint: origin xyz=0.0 0.0 0.0 rpy=0 0 0 -> xyz=0.0000 0.0000 0.0000 rpy=0 0 0
- joint Jaw: origin xyz=-0.579458 0.012806 0.011843999999999999 rpy=0 0 0 -> xyz=-57.9458 1.2806 1.1844 rpy=0 0 0
- joint RL_calf_joint: origin xyz=-0.346984 0.012964 -0.7092059999999999 rpy=0 0 0 -> xyz=-34.6984 1.2964 -70.9206 rpy=0 0 0
- joint RL_foot_fixed: origin xyz=0.030973999999999998 -0.012686999999999999 -0.454922 rpy=0 0 0 -> xyz=3.0974 -1.2687 -45.4922 rpy=0 0 0
- joint RL_hip_joint: origin xyz=0.0 0.0 0.0 rpy=0 0 0 -> xyz=-56.4942 21.9765 -79.1156 rpy=0 0 0; parent RL_pre_hip -> trunk
- joint RL_thigh_joint: origin xyz=0.0 0.0 0.0 rpy=0 0 0 -> xyz=0.0000 0.0000 0.0000 rpy=0 0 0
- joint RR_calf_joint: origin xyz=-0.448519 0.006079 -0.7266809999999999 rpy=0 0 0 -> xyz=-44.8519 0.6079 -72.6681 rpy=0 0 0
- joint RR_foot_fixed: origin xyz=-0.075565 0.033491 -0.44655 rpy=0 0 0 -> xyz=-7.5565 3.3491 -44.6550 rpy=0 0 0
- joint RR_hip_joint: origin xyz=0.0 0.0 0.0 rpy=0 0 0 -> xyz=-82.6344 -18.0470 -81.8491 rpy=0 0 0; parent RR_pre_hip -> trunk
- joint RR_thigh_joint: origin xyz=0.0 0.0 0.0 rpy=0 0 0 -> xyz=0.0000 0.0000 0.0000 rpy=0 0 0
- joint Spinal Midpoint Lower: origin xyz=-0.562901 0.01244 0.0 rpy=0 0 0 -> xyz=-56.2901 1.2440 0.0000 rpy=0 0 0
- joint Spinal Midpoint Upper: origin xyz=0.494218 -0.010922000000000001 0.0 rpy=0 0 0 -> xyz=49.4218 -1.0922 0.0000 rpy=0 0 0
- joint Start of Tail: origin xyz=-0.906485 0.020033 -0.732124 rpy=0 0 0 -> xyz=-90.6485 2.0033 -73.2124 rpy=0 0 0
- joint Top of Nose: origin xyz=0.5705129999999999 -0.012608 -0.521657 rpy=0 0 0 -> xyz=57.0513 -1.2608 -52.1657 rpy=0 0 0
- joint floating_base: origin xyz=0.0 0.0 0.0 rpy=0 0 0 -> xyz=0.0000 0.0000 0.0000 rpy=0 0 0

File: horse_like_robot.model.urdf (robot description, URDF)
Before this commit: robot a1, 28 links, 27 joints
Links:
- removed link FL_pre_hip
- removed link FR_pre_hip
- removed link RL_pre_hip
- removed link RR_pre_hip
Joints:
- removed joint FL_pre_hip_joint
- removed joint FR_pre_hip_joint
- removed joint RL_pre_hip_joint
- removed joint RR_pre_hip_joint
- joint FL_hip_joint: parent FL_pre_hip -> trunk
- joint FR_hip_joint: parent FR_pre_hip -> trunk
- joint RL_hip_joint: parent RL_pre_hip -> trunk
- joint RR_hip_joint: parent RR_pre_hip -> trunk
